File: PowerSwap.kicad_pcb (KiCad board)
At the start: 2 copper layers, 26.1 x 36.2 mm, 19 parts, among them P1 CONN_01X02, P2 CONN_01X02, U1 TPS61087

Commit message: basic track routing complete
Parts:
- moved W3 6.77 mm to (171.6, 137.2)
- moved C2 2.18 mm to (163.2, 111.2)
- moved C1 1.91 mm to (163.3, 108.3)
- moved C6 1.58 mm to (163.3, 129.0)
- moved P1 1.43 mm to (164.4, 104.8)
- moved C3 0.57 mm to (163.3, 115.7)
- moved P2 0.28 mm to (164.6, 136.8)
- moved R4 0.23 mm to (163.1, 133.5)
Routing:
- net /Vout: track 0.00 -> 27.5 mm
- net Net-(C4-Pad1): track 0.00 -> 18.5 mm, vias 0 -> 2
- net /Vin: track 11.7 -> 19.8 mm, vias 0 -> 2
- net Net-(R1-Pad1): track 0.00 -> 6.22 mm
- net Net-(C5-Pad1): track 0.00 -> 3.35 mm
- net /FB: track 6.41 -> 9.70 mm
- added copper zone on F.Cu, net /SW
- added copper zone on F.Cu, net /Vin
Other:
- net class Default: clearance 0.2 -> 0.1524
- rule solder_mask_min_width: 0.1524 -> 0.1016
- rule trace_clearance: 0.2 -> 0.1524

Commit message: completed layout and generated gerbers
Parts:
- added REF**: MountingHole_2.2mm_M2, Mounting_Holes:MountingHole_2.2mm_M2, F.Cu at (174.1, 104.8)
- added REF**: MountingHole_2.2mm_M2, Mounting_Holes:MountingHole_2.2mm_M2, F.Cu at (152.3, 104.8)
- added REF**: MountingHole_2.2mm_M2, Mounting_Holes:MountingHole_2.2mm_M2, F.Cu at (152.7, 136.5)
- added REF**: MountingHole_2.2mm_M2, Mounting_Holes:MountingHole_2.2mm_M2, F.Cu at (173.9, 136.5)
- moved W3 7.37 mm to (174.5, 130.5)
- moved C1 1.65 mm to (163.2, 110.0)
- moved C2 1.63 mm to (163.2, 112.8)
- moved R2 0.51 mm to (155.3, 119.3)
- moved W2 0.36 mm to (152.6, 116.2)
Routing:
- net /Vout: track 27.5 -> 34.7 mm
- net /FB: track 9.70 -> 10.5 mm
- added copper zone on B.Cu, net GND
Other:
- board text added: "3V<=Vin<=4.2V"
- board text added: "FB"
- board text added: "GND"
- board text added: "Vin"
- board text added: "Vout"
- board text added: "Vout = 6V Iout = 0.75A MAX"
